File: hardware/SimpleFlightController.kicad_pcb (KiCad board)
At the start: 2 copper layers, 82 parts, among them J1 Conn_01x03, J2 Screw_Terminal_01x03, J3 Conn_01x03, SW1 TS-1088-AR02016, SW2 TS-1088-AR02016, U1 TPS63070RNMR, U3 ICM-20948, U4 BME280, U5 BQ25887RGET, U6 LMR51430XDDCR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

Commit message: PCB Routing
Parts:
- moved C1 34.3 mm to (101.0, 185.5), turned to 180 degrees
- moved C14 32.8 mm to (96.5, 183.0), turned to -90 degrees
- moved L3 31.4 mm to (151.0, 170.0), turned to 180 degrees
- moved R2 31.0 mm to (266.0, 36.0)
- moved C3 30.8 mm to (222.5, 83.6)
- moved C4 30.8 mm to (222.5, 85.5)
- moved C5 30.8 mm to (222.5, 87.5)
- moved C6 30.8 mm to (222.5, 89.5)
- moved R1 28.0 mm to (262.5, 36.0)
- moved C15 28.0 mm to (154.0, 172.5)
- moved C2 23.7 mm to (224.6, 75.5)
- moved C7 23.7 mm to (224.6, 78.5)
- moved C8 23.4 mm to (108.5, 183.4), turned to -90 degrees
- moved C18 21.1 mm to (155.0, 167.5)
- moved C12 21.0 mm to (95.5, 183.0), turned to -90 degrees
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Routing:
- net +5V: track 0.00 -> 17.9 mm
- net VSYS: track 0.00 -> 9.87 mm
- net GND: track 0.00 -> 4.97 mm, vias 0 -> 2
- net Net-(U1-EN): track 0.00 -> 3.96 mm
- net Net-(U1-L1): track 0.00 -> 3.46 mm
- net Net-(U1-L2): track 0.00 -> 3.37 mm
- net Net-(U1-Vaux): track 0.00 -> 1.36 mm
- net Net-(U1-PG): track 0.00 -> 1.32 mm
