File: hardware/SimpleFlightController.kicad_pcb (KiCad board)
At the start: 2 copper layers, 82 parts, among them J1 Conn_01x03, J2 Screw_Terminal_01x03, J3 Conn_01x03, SW1 TS-1088-AR02016, SW2 TS-1088-AR02016, U1 TPS63070RNMR, U3 ICM-20948, U4 BME280, U5 BQ25887RGET, U6 LMR51430XDDCR, U7 STM32F722RETx, X1 X322525MOB4SI, X2 Q13FC1350000400

Commit message: Finishing Touches
Parts:
- moved R1 144.7 mm to (139.6, 112.4), turned to 180 degrees
- moved R2 144.3 mm to (143.6, 112.4)
- moved USB1 144.3 mm to (141.6, 115.8)
- moved C37 143.5 mm to (127.8, 91.3), turned to -135 degrees
- moved X1 143.2 mm to (126.0, 89.5), turned to -45 degrees
- moved C38 142.8 mm to (124.2, 87.7), turned to 45 degrees
- moved X2 142.0 mm to (130.5, 84.0), turned to -135 degrees
- moved C35 141.1 mm to (131.2, 86.1), turned to -45 degrees
- moved SW2 140.4 mm to (123.3, 75.0), turned to -90 degrees
- moved SW1 139.9 mm to (127.5, 75.0), turned to -90 degrees
- moved C36 138.2 mm to (132.6, 84.7), turned to -45 degrees
- moved R24 135.4 mm to (123.2, 78.6), turned to -90 degrees
- moved C39 134.1 mm to (127.7, 79.1), turned to 90 degrees
- moved C21 118.9 mm to (126.4, 108.4)
- moved C24 118.9 mm to (126.4, 111.4)
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Routing:
- net GND: track 4.97 -> 303.3 mm, vias 2 -> 31
- net +3.3V: track 0.00 -> 122.0 mm
- net /BOOT: track 0.00 -> 73.3 mm, vias 0 -> 2
- net /SERVO1: track 0.00 -> 59.1 mm, vias 0 -> 2
- net Net-(U5-BTST): track 0.00 -> 50.3 mm, vias 0 -> 2
- net /I2C_SCL: track 0.00 -> 41.9 mm, vias 0 -> 2
- net /SERVO2: track 0.00 -> 41.8 mm, vias 0 -> 2
- net /I2C_SDA: track 0.00 -> 40.7 mm, vias 0 -> 2
- net Net-(U7-VCAP_1): track 0.00 -> 40.6 mm, vias 0 -> 2
- net /MID: track 0.00 -> 34.7 mm, vias 0 -> 3
- net /BQ_INT: track 0.00 -> 34.0 mm, vias 0 -> 2
- net /SD_DAT0: track 0.00 -> 32.5 mm, vias 0 -> 2
- net +BAT: track 0.00 -> 29.2 mm, vias 0 -> 1
- net /SD_DAT1: track 0.00 -> 28.9 mm, vias 0 -> 2
- net VBUS: track 0.00 -> 27.5 mm, vias 0 -> 4
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- added copper zone on B.Cu, net GND
- added copper zone on F.Cu, net GND
Other:
- board outline added: 50 x 55 mm

Commit message: Final Touches
Other:
- board text added: "SIMPLE FLIGHT CONTROLLER @FREEDOM"
- board text added: "SIMPLE FLIGHT CONTROLLER @Freedom"
Changed lines of the file:
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@@
 			)
 		)
-		(pad "" thru_hole circle
+		(pad "" np_thru_hole circle
 			(at -2.89 -1.3)
 			(size 0.7 0.7)
 			(drill 0.7)
 			(layers "*.Cu" "*.Mask")
-			(remove_unused_layers no)
-		)
-		(pad "" thru_hole circle
+		)
+		(pad "" np_thru_hole circle
 			(at 2.89 -1.3)
 			(size 0.7 0.7)
 			(drill 0.7)
 			(layers "*.Cu" "*.Mask")
-			(remove_unused_layers no)
 		)
 		(pad "13" thru_hole oval
@@
 		(layer "Edge.Cuts")
 	)
+	(gr_text "SIMPLE FLIGHT CONTROLLER\n@Freedom"
+		(at 168.5 101.5 90)
+		(layer "B.Cu")
+		(effects
+			(font
+				(size 1.5 1.5)
+				(thickness 0.3)
+				(bold yes)
+			)
+			(justify left bottom)
+		)
+	)
+	(gr_text "SIMPLE FLIGHT CONTROLLER\n@FREEDOM"
+		(at 168.5 99 90)
+		(layer "F.SilkS")
+		(effects
+			(font
+				(size 1.5 1.5)
+				(thickness 0.3)
+				(bold yes)
+			)
+			(justify left bottom)
+		)
+	)
 	(segment
