File: hardware/_restore_backup_2026-06-08T18-18-01-208/SimpleFlightController.kicad_pcb (KiCad board)
At the start: 2 copper layers, 82 parts, among them J1 Conn_01x03, J2 Screw_Terminal_01x03, J3 Conn_01x03, SW1 TS-1088-AR02016, SW2 TS-1088-AR02016, U1 TPS63070RNMR, U3 ICM-20948, U4 BME280, U5 BQ25887RGET, U6 LMR51430XDDCR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

Commit message: PCB Layout Almost Final
Parts:
- moved C26 143.5 mm to (26.5, 27.0), turned to 0 degrees
- moved C34 136.7 mm to (29.4, 27.0), turned to 0 degrees
- moved C32 132.5 mm to (26.5, 38.8), turned to 0 degrees
- moved C31 131.7 mm to (26.5, 36.9)
- moved C30 126.0 mm to (26.5, 34.9)
- moved C33 124.4 mm to (29.4, 25.0), turned to 0 degrees
- moved C27 121.1 mm to (26.5, 29.0), turned to 0 degrees
- moved C29 119.8 mm to (26.5, 32.9), turned to 0 degrees
- moved C28 119.7 mm to (26.5, 30.9), turned to 0 degrees
- moved R21 43.5 mm to (49.3, 134.3), turned to 0 degrees
- moved R20 39.3 mm to (49.3, 132.5), turned to 0 degrees
- moved R23 37.4 mm to (51.7, 125.5), turned to 0 degrees
- moved R19 35.5 mm to (49.3, 130.8), turned to 0 degrees
- moved R22 34.4 mm to (51.7, 123.8), turned to 0 degrees
- moved R18 32.8 mm to (49.3, 129.0), turned to 0 degrees
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